File: STOP!Timer/LCD_DRIVER.kicad_sch (KiCad schematic)
At the start: 5 parts, among them J2 Conn_01x16_Socket, Q1 2N2219, U4 PCF8574

Commit message: Update Schematic
Parts:
- removed Q1: 2N2219, Package_TO_SOT_THT:TO-39-3, symbol Transistor_BJT:2N2219
- removed R1: R, symbol Device:R
- added DS1: HY1602E, Display:WC1602A, symbol Display_Character:WC1602A
- added Q1: AO3401A, Package_TO_SOT_SMD:SOT-23, symbol Transistor_FET:AO3401A
- U4: footprint (none) -> Package_SO:SSOP-20_4.4x6.5mm_P0.65mm; JLC (none) -> C57790
Connections:
- net GND: now also DS1.1 (VSS), Q1.2 (S)
- net LCD_BACKLIGHT_ENABLE: now also Q1.1 (G)
- net LCD_DB4: now also DS1.11 (D4)
- net LCD_DB5: now also DS1.12 (D5)
- net LCD_DB6: now also DS1.13 (D6)
- net LCD_DB7: now also DS1.14 (D7)
- net LCD_E: now also DS1.6 (E)
- net LCD_RS: now also DS1.4 (RS)
- net LCD_RW: now also DS1.5 (R/W)
- net VCC: now also DS1.15 (LED(+)), DS1.2 (VDD), DS1.3 (VO)
- new net: DS1.16 (LED(-)), Q1.3 (D)
- no-connect marks 4 -> 8

Commit message: Update 31 03 2026
Parts:
- removed J2: Conn_01x16_Socket, symbol Connector:Conn_01x16_Socket
- added JP1: SolderJumper_2_Bridged, Jumper:SolderJumper-2_P1.3mm_Bridged_Pad1.0x1.5mm, symbol Jumper:SolderJumper_2_Bridged
- RV1: value 10k - 20k -> 20k; footprint (none) -> Potentiometer_THT:Potentiometer_Bourns_3386W_Horizontal
Connections:
- net LCD_BACKLIGHT_ENABLE: now also JP1.1 (A)
- net LCD_CONTRAST: now also DS1.3 (VO)
- net VCC: no longer DS1.3 (VO)
- net LCD_BT: no longer names the net of U4.7 (P3)
- net LCD_BT: now also JP1.2 (B)
Other:
- note removed: "2004 or 1602 Display Port"
- moved on the sheet: RV1

Commit message: update to order version 1.0
Parts:
- RV1: JLC (none) -> C221841
Changed lines of the file:
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@@
+			)
+		)
+		(property "JLC" "C221841"
+			(at 233.68 69.85 0)
+			(effects
+				(font
+					(size 1.27 1.27)
+				)
+				(hide yes)
 			)
 		)

Commit message: Update
Parts:
- RV1: value 20k -> 20k
